File: hardware/v1.0/led-matrix.kicad_pcb (KiCad board)
At the start: 2 copper layers, 40 x 40 mm, 93 parts, among them J1 Conn_01x01, J10 Conn_01x01, J11 Conn_01x01, J12 Conn_01x01, J2 Conn_01x01, J3 Conn_01x01, J4 Conn_01x01, J5 Conn_01x01, J6 Conn_01x01, J7 Conn_01x01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

Commit message: hardware done.
- update pcb.

Signed-off-by: UnsicentificLaLaLaLa <zhaohao1997@foxmail.com>
Parts:
- R1, R2, R3, R4, R5, R6, R7, R8: value 1K -> 2K
- TP1, TP2, TP3: moved to B.Cu
- moved TP1 23.8 mm to (77.5, 57.5), turned to 180 degrees
- moved TP3 20.2 mm to (75.0, 57.5), turned to 180 degrees
- moved TP2 19.5 mm to (80.0, 57.5), turned to 180 degrees
- moved J1 10.0 mm to (46.0, 40.0)
- moved J10 10.0 mm to (84.0, 40.0)
- moved J11 10.0 mm to (84.0, 30.0)
- moved J2 10.0 mm to (46.0, 30.0)
- moved J4 10.0 mm to (84.0, 40.0)
- moved J5 10.0 mm to (84.0, 30.0)
- moved J7 10.0 mm to (46.0, 40.0)
- moved J8 10.0 mm to (46.0, 30.0)
- turned D1 to -135 degrees
- turned D17 to -135 degrees
- turned D18 to -45 degrees
- turned D19 to -135 degrees
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Connections:
- D13 pad 1: /PA14 -> /PA15
- D14 pad 1: /PA13 -> /PA2
- D15 pad 1: /PA15 -> /PA14
- D16 pad 1: /PA2 -> /PA13
- D21 pad 1: /PA14 -> /PA15
- D22 pad 1: /PA13 -> /PA2
- D23 pad 1: /PA15 -> /PA14
- D24 pad 1: /PA2 -> /PA13
- D29 pad 1: /PA14 -> /PA15
- D30 pad 1: /PA13 -> /PA2
- D31 pad 1: /PA15 -> /PA14
- D32 pad 1: /PA2 -> /PA13
- D37 pad 1: /PA14 -> /PA15
- D38 pad 1: /PA13 -> /PA2
- D39 pad 1: /PA15 -> /PA14
- D40 pad 1: /PA2 -> /PA13
- D45 pad 1: /PA14 -> /PA15
- D46 pad 1: /PA13 -> /PA2
- D47 pad 1: /PA15 -> /PA14
- D48 pad 1: /PA2 -> /PA13
- D5 pad 1: /PA14 -> /PA15
- D53 pad 1: /PA14 -> /PA15
- D54 pad 1: /PA13 -> /PA2
- D55 pad 1: /PA15 -> /PA14
- D56 pad 1: /PA2 -> /PA13
- D6 pad 1: /PA13 -> /PA2
- D61 pad 1: /PA14 -> /PA15
- D62 pad 1: /PA13 -> /PA2
- D63 pad 1: /PA15 -> /PA14
- D64 pad 1: /PA2 -> /PA13
- D7 pad 1: /PA15 -> /PA14
- D8 pad 1: /PA2 -> /PA13
Routing:
- net GND: track 7.20 -> 65.6 mm, vias 3 -> 59
- net /PA14: track 80.8 -> 62.9 mm
- net /PA2: track 68.9 -> 56.3 mm, vias 8 -> 11
- net VCC: track 66.2 -> 55.6 mm
- net /PA13: track 84.4 -> 74.6 mm
- net /PA15: track 63.5 -> 54.9 mm, vias 9 -> 11
- net /PA9: track 22.0 -> 15.7 mm, vias 4 -> 2
- net /PA5: track 14.5 -> 20.8 mm, vias 2 -> 4
- net /PA10: track 15.7 -> 21.5 mm, vias 2 -> 4
- net /PA12: track 28.0 -> 22.5 mm
- net /PA0: track 68.4 -> 72.9 mm, vias 11 -> 10
- net Net-(D17-A): track 33.9 -> 37.7 mm, vias 2 -> 0
- net /PA6: track 19.7 -> 16.0 mm
- net /PA11: track 23.2 -> 20.1 mm
- net /PA7: track 17.6 -> 20.3 mm, vias 4 -> 2
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- added copper zone on B.Cu, net GND
- added copper zone on F.Cu, net GND
Other:
- board text added: "C"
- board text added: "D"
- board text added: "DIN"
- board text added: "DOUT"
- board text added: "G"
- board text added: "GND"
- board text added: "VCC"

Commit message: add production.
- add prd.
- update pcb file.

Signed-off-by: zhaohao <zhaohao@mindmotion.com.cn>
Parts:
- U1: value MM32G0001A1T -> MM32G0001A1N
Other:
- board text added: "JLCJLCJLCJLC"
- board text added: "led-matrix v1.0"
Changed lines of the file:
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@@
         (effects (font (size 1 1) (thickness 0.15)))
     )
-    (fp_text value "MM32G0001A1T" (at 0 2.82 45) (layer "F.Fab")
+    (fp_text value "MM32G0001A1N" (at 0 2.82 45) (layer "F.Fab")
         (effects (font (size 1 1) (thickness 0.15)))
     )
@@
     (effects (font (size 1 0.8) (thickness 0.15)) (justify right mirror))
   )
+  (gr_text "led-matrix v1.0" (at 73.406 56.896) (layer "B.SilkS")
+    (effects (font (size 0.8 0.8) (thickness 0.15)) (justify left mirror))
+  )
   (gr_text "C" (at 77.5 56) (layer "B.SilkS")
     (effects (font (size 1 1) (thickness 0.15)) (justify mirror))
@@
     (effects (font (size 1 0.8) (thickness 0.15)) (justify left mirror))
   )
+  (gr_text "JLCJLCJLCJLC" (at 73.406 58.166) (layer "B.SilkS")
+    (effects (font (size 0.8 0.6) (thickness 0.15)) (justify left mirror))
+  )
   (gr_text "D" (at 80 56) (layer "B.SilkS")
